Commit message: added new tri-snake robot; added layer connections for nearest layers

File: resources/3D/urdf/tri-snake.urdf (robot description, URDF)
Before this commit: robot tri-snake, 10 links, 9 joints
Links:
- link base: geometry visual box size=6 5 2.6
- link body1: geometry visual box size=4.6 3.7 1.6
- link body2: geometry visual box size=4.6 1.4 3.3
- link body3: geometry visual box size=4.6 3.4 1.16
- link body4: geometry visual box size=4.6 2.27 1.4
- link body5: geometry visual box size=4.6 1.7 2.4
- link body6: geometry visual box size=4.6 2.7 1.4
- link body7: geometry visual box size=3.5 2.7 4.6
- link body8: geometry visual box size=1.2 2.7 4.6
- link body9: geometry visual box size=3.5 2.7 4.6
Joints:
- joint body1_to_base: origin xyz=9.5 0 0 rpy=0 0 0 -> xyz=5.5 0 0 rpy=0 0 0
- joint body2_to_body1: origin xyz=14.2 0 0 rpy=0 0 0 -> xyz=8.2 0 0 rpy=0 0 0
- joint body3_to_body2: origin xyz=14.2 0 0 rpy=0 0 0 -> xyz=8.2 0 0 rpy=0 0 0
- joint body4_to_base: origin xyz=-9.5 0 0 rpy=0 0 0 -> xyz=-5.5 0 0 rpy=0 0 0
- joint body5_to_body4: origin xyz=-14.2 0 0 rpy=0 0 0 -> xyz=-8.2 0 0 rpy=0 0 0
- joint body6_to_body5: origin xyz=-14.2 0 0 rpy=0 0 0 -> xyz=-8.2 0 0 rpy=0 0 0
- joint body7_to_base: origin xyz=0 0 3.5 rpy=0 0 0 -> xyz=0 0 2.1 rpy=0 0 0
- joint body8_to_body7: origin xyz=0 0 14.2 rpy=0 0 0 -> xyz=0 0 8.2 rpy=0 0 0
- joint body9_to_body8: origin xyz=0 0 14.2 rpy=0 0 0 -> xyz=0 0 8.2 rpy=0 0 0

File: resources/3D/urdf/tri-snake.xacro (robot description, xacro)
@@ -1,7 +1,7 @@
 <?xml version="1.0"?>
 <robot xmlns:xacro="http://www.ros.org/wiki/xacro" name="tri-snake">
-  <xacro:property name="baselen" value="10"/>
-  <xacro:property name="baseheight" value="4"/>
-  <xacro:property name="bodylen" value="7.6"/>
+  <xacro:property name="baselen" value="6"/>
+  <xacro:property name="baseheight" value="2.6"/>
+  <xacro:property name="bodylen" value="4.6"/>
   <xacro:property name="joint_offset" value="0.5"/>
   <material name="blue">
@@ -14,5 +14,5 @@
     <visual>
       <geometry>
-        <box size="10 5 4"/>
+        <box size="${baselen} 5 ${baseheight}"/>
       </geometry>
       <material name="green"/>
@@ -30,5 +30,5 @@
     <visual>
       <geometry>
-        <box size="7.6 4.7 2.6"/>
+        <box size="${bodylen} 3.7 1.6"/>
       </geometry>
       <origin rpy="0 0 0" xyz="${bodylen-joint_offset} 0 0"/>
@@ -46,5 +46,5 @@
     <visual>
       <geometry>
-        <box size="7.6 2.4 5.3"/>
+        <box size="${bodylen} 1.4 3.3"/>
       </geometry>
       <origin rpy="0 0 0" xyz="${bodylen-joint_offset} 0 0"/>
@@ -62,5 +62,5 @@
     <visual>
       <geometry>
-        <box size="7.6 6.4 2.16"/>
+        <box size="${bodylen} 3.4 1.16"/>
       </geometry>
       <origin rpy="0 0 0" xyz="${bodylen-joint_offset} 0 0"/>
@@ -79,5 +79,5 @@
     <visual>
       <geometry>
-        <box size="7.6 3.27 1.4"/>
+        <box size="${bodylen} 2.27 1.4"/>
       </geometry>
       <origin rpy="0 0 0" xyz="${-(bodylen-joint_offset)} 0 0"/>
@@ -95,5 +95,5 @@
     <visual>
       <geometry>
-        <box size="7.6 2.7 4.4"/>
+        <box size="${bodylen} 1.7 2.4"/>
       </geometry>
       <origin rpy="0 0 0" xyz="${-(bodylen-joint_offset)} 0 0"/>
@@ -111,5 +111,5 @@
     <visual>
       <geometry>
-        <box size="7.6 4.7 2.4"/>
+        <box size="${bodylen} 2.7 1.4"/>
       </geometry>
       <origin rpy="0 0 0" xyz="${-(bodylen-joint_offset)} 0 0"/>
@@ -128,5 +128,5 @@
     <visual>
       <geometry>
-        <box size="3.5 4.7 7.6"/>
+        <box size="3.5 2.7 ${bodylen}"/>
       </geometry>
       <origin rpy="0 0 0" xyz="0 0 ${bodylen-joint_offset} "/>
@@ -144,5 +144,5 @@
     <visual>
       <geometry>
-        <box size="1.2 4.7 7.6"/>
+        <box size="1.2 2.7 ${bodylen}"/>
       </geometry>
       <origin rpy="0 0 0" xyz="0 0 ${bodylen-joint_offset}"/>
@@ -160,5 +160,5 @@
     <visual>
       <geometry>
-        <box size="6.5 4.7 7.6"/>
+        <box size="3.5 2.7 ${bodylen}"/>
       </geometry>
       <origin rpy="0 0 0" xyz="0 0 ${bodylen-joint_offset}"/>
