Commit message: fixed bug for selecting nearest C-layer; changed config for snake robot

File: resources/3D/urdf/snake.urdf (robot description, URDF)
Before this commit: robot snake, 4 links, 3 joints
Links:
- link base: geometry visual box size=7.5 5 2.8
- link body1: geometry visual box size=4.6 3.7 1.6
- link body2: geometry visual box size=4.6 1.4 3.3
- link body3: geometry visual box size=4.6 3.4 1.16
Joints:
- joint body1_to_base: limit lower=-1.0471975512 upper=1.0471975512 effort=100 velocity=5 -> lower=-1.57079632679 upper=1.57079632679 effort=100 velocity=5; origin xyz=9.5 0 0 rpy=0 0 0 -> xyz=7.0 0 0 rpy=0 0 0
- joint body2_to_body1: limit lower=-0.785398163397 upper=0.785398163397 effort=100 velocity=5 -> lower=-1.57079632679 upper=1.57079632679 effort=100 velocity=5; origin xyz=14.2 0 0 rpy=0 0 0 -> xyz=8.2 0 0 rpy=0 0 0
- joint body3_to_body2: origin xyz=14.2 0 0 rpy=0 0 0 -> xyz=8.2 0 0 rpy=0 0 0

File: resources/3D/urdf/snake.xacro (robot description, xacro)
@@ -1,6 +1,7 @@
 <?xml version="1.0"?>
-<robot xmlns:xacro="http://www.ros.org/wiki/xacro" name="snake">
-  <xacro:property name="baselen" value="10"/>
-  <xacro:property name="bodylen" value="7.6"/>
+<robot xmlns:xacro="http://www.ros.org/wiki/xacro" name="tri-snake">
+  <xacro:property name="baselen" value="7.5"/>
+  <xacro:property name="baseheight" value="2.8"/>
+  <xacro:property name="bodylen" value="4.6"/>
   <xacro:property name="joint_offset" value="0.5"/>
   <material name="blue">
@@ -13,9 +14,10 @@
     <visual>
       <geometry>
-        <box size="10 5 4"/>
+        <box size="${baselen} 5 ${baseheight}"/>
       </geometry>
       <material name="green"/>
     </visual>
   </link>
+  <!-- First chain -->
   <joint name="body1_to_base" type="revolute">
     <parent link="base"/>
@@ -23,10 +25,10 @@
     <origin rpy="0 0 0" xyz="${baselen-joint_offset} 0 0"/>
     <axis xyz="0 1 0"/>
-    <limit lower="${-pi/3}" upper="${pi/3}" effort="100" velocity="5"/>
+    <limit lower="${-pi/2}" upper="${pi/2}" effort="100" velocity="5"/>
   </joint>
   <link name="body1">
     <visual>
       <geometry>
-        <box size="7.6 4.7 2.4"/>
+        <box size="${bodylen} 3.7 1.6"/>
       </geometry>
       <origin rpy="0 0 0" xyz="${bodylen-joint_offset} 0 0"/>
@@ -39,10 +41,10 @@
     <origin rpy="0 0 0" xyz="${bodylen*2-joint_offset*2} 0 0"/>
     <axis xyz="0 0 1"/>
-    <limit lower="${-pi/4}" upper="${pi/4}" effort="100" velocity="5"/>
+    <limit lower="${-pi/2}" upper="${pi/2}" effort="100" velocity="5"/>
   </joint>
   <link name="body2">
     <visual>
       <geometry>
-        <box size="7.6 4.7 2.4"/>
+        <box size="${bodylen} 1.4 3.3"/>
       </geometry>
       <origin rpy="0 0 0" xyz="${bodylen-joint_offset} 0 0"/>
@@ -60,5 +62,5 @@
     <visual>
       <geometry>
-        <box size="7.6 4.7 2.4"/>
+        <box size="${bodylen} 3.4 1.16"/>
       </geometry>
       <origin rpy="0 0 0" xyz="${bodylen-joint_offset} 0 0"/>

Commit message: Changed urdf from tri-snake to tree

File: resources/3D/urdf/snake.urdf (robot description, URDF)
Before this commit: robot tri-snake, 4 links, 3 joints
Joints:
- joint body1_to_base: limit lower=-1.57079632679 upper=1.57079632679 effort=100 velocity=5 -> lower=-1.5707963267948966 upper=1.5707963267948966 effort=100 velocity=5
- joint body2_to_body1: limit lower=-1.57079632679 upper=1.57079632679 effort=100 velocity=5 -> lower=-1.5707963267948966 upper=1.5707963267948966 effort=100 velocity=5
- joint body3_to_body2: limit lower=-1.57079632679 upper=1.57079632679 effort=100 velocity=5 -> lower=-1.5707963267948966 upper=1.5707963267948966 effort=100 velocity=5

File: resources/3D/urdf/snake.xacro (robot description, xacro)
@@ -1,4 +1,4 @@
 <?xml version="1.0"?>
-<robot xmlns:xacro="http://www.ros.org/wiki/xacro" name="tri-snake">
+<robot xmlns:xacro="http://www.ros.org/wiki/xacro" name="snake">
   <xacro:property name="baselen" value="7.5"/>
   <xacro:property name="baseheight" value="2.8"/>

File: resources/3D/urdf/tree.urdf (robot description, URDF)
Before this commit: robot tri-snake, 10 links, 9 joints
Links:
- link base: geometry visual box size=6 5 2.6
- link body1: geometry visual box size=4.6 3.7 1.6
- link body2: geometry visual box size=4.6 1.4 3.3
- link body3: geometry visual box size=4.6 3.4 1.16
- link body4: geometry visual box size=4.6 2.27 1.4
- link body5: geometry visual box size=4.6 1.7 2.4
- link body6: geometry visual box size=4.6 2.7 1.4
- link body7: geometry visual box size=3.5 2.7 4.6
- link body8: geometry visual box size=1.2 2.7 4.6
- link body9: geometry visual box size=3.5 2.7 4.6
Joints:
- joint body1_to_base: limit lower=${-pi/2} upper=${pi/2} effort=100 velocity=5 -> lower=-1.5707963267948966 upper=1.5707963267948966 effort=100 velocity=5; origin xyz=${baselen-joint_offset} 0 0 rpy=0 0 0 -> xyz=5.5 0 0 rpy=0 0 0
- joint body2_to_body1: limit lower=${-pi/2} upper=${pi/2} effort=100 velocity=5 -> lower=-1.5707963267948966 upper=1.5707963267948966 effort=100 velocity=5; origin xyz=${bodylen*2-joint_offset*2} 0 0 rpy=0 0 0 -> xyz=8.2 0 0 rpy=0 0 0
- joint body3_to_body2: limit lower=${-pi/2} upper=${pi/2} effort=100 velocity=5 -> lower=-1.5707963267948966 upper=1.5707963267948966 effort=100 velocity=5; origin xyz=${bodylen*2-joint_offset*2} 0 0 rpy=0 0 0 -> xyz=8.2 0 0 rpy=0 0 0
- joint body4_to_base: limit lower=${-pi/2} upper=${pi/2} effort=100 velocity=5 -> lower=-1.5707963267948966 upper=1.5707963267948966 effort=100 velocity=5; origin xyz=${-(baselen-joint_offset)} 0 0 rpy=0 0 0 -> xyz=-5.5 0 0 rpy=0 0 0
- joint body5_to_body4: limit lower=${-pi/2} upper=${pi/2} effort=100 velocity=5 -> lower=-1.5707963267948966 upper=1.5707963267948966 effort=100 velocity=5; origin xyz=${-(bodylen*2-joint_offset*2)} 0 0 rpy=0 0 0 -> xyz=-8.2 0 0 rpy=0 0 0
- joint body6_to_body5: limit lower=${-pi/2} upper=${pi/2} effort=100 velocity=5 -> lower=-1.5707963267948966 upper=1.5707963267948966 effort=100 velocity=5; origin xyz=${-(bodylen*2-joint_offset*2)} 0 0 rpy=0 0 0 -> xyz=-8.2 0 0 rpy=0 0 0
- joint body7_to_base: limit lower=${-pi/2} upper=${pi/2} effort=100 velocity=5 -> lower=-1.5707963267948966 upper=1.5707963267948966 effort=100 velocity=5; origin xyz=0 0 ${baseheight-joint_offset} rpy=0 0 0 -> xyz=0 0 2.1 rpy=0 0 0
- joint body8_to_body7: limit lower=${-pi/2} upper=${pi/2} effort=100 velocity=5 -> lower=-1.5707963267948966 upper=1.5707963267948966 effort=100 velocity=5; origin xyz=0 0 ${bodylen*2-joint_offset*2} rpy=0 0 0 -> xyz=0 0 8.2 rpy=0 0 0
- joint body9_to_body8: limit lower=${-pi/2} upper=${pi/2} effort=100 velocity=5 -> lower=-1.5707963267948966 upper=1.5707963267948966 effort=100 velocity=5; origin xyz=0 0 ${bodylen*2-joint_offset*2} rpy=0 0 0 -> xyz=0 0 8.2 rpy=0 0 0

File: resources/3D/urdf/tree.xacro (robot description, xacro)
@@ -1,8 +1,8 @@
-<?xml version="1.0" ?>
-<!-- =================================================================================== -->
-<!-- |    This document was autogenerated by xacro from tri-snake.xacro                | -->
-<!-- |    EDITING THIS FILE BY HAND IS NOT RECOMMENDED                                 | -->
-<!-- =================================================================================== -->
-<robot name="tri-snake" xmlns:xacro="http://www.ros.org/wiki/xacro">
+<?xml version="1.0"?>
+<robot xmlns:xacro="http://www.ros.org/wiki/xacro" name="tree">
+  <xacro:property name="baselen" value="6"/>
+  <xacro:property name="baseheight" value="2.6"/>
+  <xacro:property name="bodylen" value="4.6"/>
+  <xacro:property name="joint_offset" value="0.5"/>
   <material name="blue">
     <color rgba="0 0 0.8 0.7"/>
@@ -14,5 +14,5 @@
     <visual>
       <geometry>
-        <box size="6 5 2.6"/>
+        <box size="${baselen} 5 ${baseheight}"/>
       </geometry>
       <material name="green"/>
@@ -23,14 +23,14 @@
     <parent link="base"/>
     <child link="body1"/>
-    <origin rpy="0 0 0" xyz="5.5 0 0"/>
+    <origin rpy="0 0 0" xyz="${baselen-joint_offset} 0 0"/>
     <axis xyz="0 1 0"/>
-    <limit effort="100" lower="-1.57079632679" upper="1.57079632679" velocity="5"/>
+    <limit lower="${-pi/2}" upper="${pi/2}" effort="100" velocity="5"/>
   </joint>
   <link name="body1">
     <visual>
       <geometry>
-        <box size="4.6 3.7 1.6"/>
+        <box size="${bodylen} 3.7 1.6"/>
       </geometry>
-      <origin rpy="0 0 0" xyz="4.1 0 0"/>
+      <origin rpy="0 0 0" xyz="${bodylen-joint_offset} 0 0"/>
       <material name="blue"/>
     </visual>
@@ -39,14 +39,14 @@
     <parent link="body1"/>
     <child link="body2"/>
-    <origin rpy="0 0 0" xyz="8.2 0 0"/>
+    <origin rpy="0 0 0" xyz="${bodylen*2-joint_offset*2} 0 0"/>
     <axis xyz="0 0 1"/>
-    <limit effort="100" lower="-1.57079632679" upper="1.57079632679" velocity="5"/>
+    <limit lower="${-pi/2}" upper="${pi/2}" effort="100" velocity="5"/>
   </joint>
   <link name="body2">
     <visual>
       <geometry>
-        <box size="4.6 1.4 3.3"/>
+        <box size="${bodylen} 1.4 3.3"/>
       </geometry>
-      <origin rpy="0 0 0" xyz="4.1 0 0"/>
+      <origin rpy="0 0 0" xyz="${bodylen-joint_offset} 0 0"/>
       <material name="blue"/>
     </visual>
@@ -55,14 +55,14 @@
     <parent link="body2"/>
     <child link="body3"/>
-    <origin rpy="0 0 0" xyz="8.2 0 0"/>
+    <origin rpy="0 0 0" xyz="${bodylen*2-joint_offset*2} 0 0"/>
     <axis xyz="0 1 0"/>
-    <limit effort="100" lower="-1.57079632679" upper="1.57079632679" velocity="5"/>
+    <limit lower="${-pi/2}" upper="${pi/2}" effort="100" velocity="5"/>
   </joint>
   <link name="body3">
     <visual>
       <geometry>
-        <box size="4.6 3.4 1.16"/>
+        <box size="${bodylen} 3.4 1.16"/>
       </geometry>
-      <origin rpy="0 0 0" xyz="4.1 0 0"/>
+      <origin rpy="0 0 0" xyz="${bodylen-joint_offset} 0 0"/>
       <material name="blue"/>
     </visual>
@@ -72,14 +72,14 @@
     <parent link="base"/>
     <child link="body4"/>
-    <origin rpy="0 0 0" xyz="-5.5 0 0"/>
+    <origin rpy="0 0 0" xyz="${-(baselen-joint_offset)} 0 0"/>
     <axis xyz="0 1 0"/>
-    <limit effort="100" lower="-1.57079632679" upper="1.57079632679" velocity="5"/>
+    <limit lower="${-pi/2}" upper="${pi/2}" effort="100" velocity="5"/>
   </joint>
   <link name="body4">
     <visual>
       <geometry>
-        <box size="4.6 2.27 1.4"/>
+        <box size="${bodylen} 2.27 1.4"/>
       </geometry>
-      <origin rpy="0 0 0" xyz="-4.1 0 0"/>
+      <origin rpy="0 0 0" xyz="${-(bodylen-joint_offset)} 0 0"/>
       <material name="blue"/>
     </visual>
@@ -88,14 +88,14 @@
     <parent link="body4"/>
     <child link="body5"/>
-    <origin rpy="0 0 0" xyz="-8.2 0 0"/>
+    <origin rpy="0 0 0" xyz="${-(bodylen*2-joint_offset*2)} 0 0"/>
     <axis xyz="0 0 1"/>
-    <limit effort="100" lower="-1.57079632679" upper="1.57079632679" velocity="5"/>
+    <limit lower="${-pi/2}" upper="${pi/2}" effort="100" velocity="5"/>
   </joint>
   <link name="body5">
     <visual>
       <geometry>
-        <box size="4.6 1.7 2.4"/>
+        <box size="${bodylen} 1.7 2.4"/>
       </geometry>
-      <origin rpy="0 0 0" xyz="-4.1 0 0"/>
+      <origin rpy="0 0 0" xyz="${-(bodylen-joint_offset)} 0 0"/>
       <material name="blue"/>
     </visual>
@@ -104,14 +104,14 @@
     <parent link="body5"/>
     <child link="body6"/>
-    <origin rpy="0 0 0" xyz="-8.2 0 0"/>
+    <origin rpy="0 0 0" xyz="${-(bodylen*2-joint_offset*2)} 0 0"/>
     <axis xyz="0 1 0"/>
-    <limit effort="100" lower="-1.57079632679" upper="1.57079632679" velocity="5"/>
+    <limit lower="${-pi/2}" upper="${pi/2}" effort="100" velocity="5"/>
   </joint>
   <link name="body6">
     <visual>
       <geometry>
-        <box size="4.6 2.7 1.4"/>
+        <box size="${bodylen} 2.7 1.4"/>
       </geometry>
-      <origin rpy="0 0 0" xyz="-4.1 0 0"/>
+      <origin rpy="0 0 0" xyz="${-(bodylen-joint_offset)} 0 0"/>
       <material name="blue"/>
     </visual>
@@ -121,14 +121,14 @@
     <parent link="base"/>
     <child link="body7"/>
-    <origin rpy="0 0 0" xyz="0 0 2.1"/>
+    <origin rpy="0 0 0" xyz="0 0 ${baseheight-joint_offset}"/>
     <axis xyz="1 0 0"/>
-    <limit effort="100" lower="-1.57079632679" upper="1.57079632679" velocity="5"/>
+    <limit lower="${-pi/2}" upper="${pi/2}" effort="100" velocity="5"/>
   </joint>
   <link name="body7">
     <visual>
       <geometry>
-        <box size="3.5 2.7 4.6"/>
+        <box size="3.5 2.7 ${bodylen}"/>
       </geometry>
-      <origin rpy="0 0 0" xyz="0 0 4.1 "/>
+      <origin rpy="0 0 0" xyz="0 0 ${bodylen-joint_offset} "/>
       <material name="blue"/>
     </visual>
@@ -137,14 +137,14 @@
     <parent link="body7"/>
     <child link="body8"/>
-    <origin rpy="0 0 0" xyz="0 0 8.2"/>
+    <origin rpy="0 0 0" xyz="0 0 ${bodylen*2-joint_offset*2}"/>
     <axis xyz="0 1 0"/>
-    <limit effort="100" lower="-1.57079632679" upper="1.57079632679" velocity="5"/>
+    <limit lower="${-pi/2}" upper="${pi/2}" effort="100" velocity="5"/>
   </joint>
   <link name="body8">
     <visual>
       <geometry>
-        <box size="1.2 2.7 4.6"/>
+        <box size="1.2 2.7 ${bodylen}"/>
       </geometry>
-      <origin rpy="0 0 0" xyz="0 0 4.1"/>
+      <origin rpy="0 0 0" xyz="0 0 ${bodylen-joint_offset}"/>
       <material name="blue"/>
     </visual>
@@ -153,14 +153,14 @@
     <parent link="body8"/>
     <child link="body9"/>
-    <origin rpy="0 0 0" xyz="0 0 8.2"/>
+    <origin rpy="0 0 0" xyz="0 0 ${bodylen*2-joint_offset*2}"/>
     <axis xyz="1 0 0"/>
-    <limit effort="100" lower="-1.57079632679" upper="1.57079632679" velocity="5"/>
+    <limit lower="${-pi/2}" upper="${pi/2}" effort="100" velocity="5"/>
   </joint>
   <link name="body9">
     <visual>
       <geometry>
-        <box size="3.5 2.7 4.6"/>
+        <box size="3.5 2.7 ${bodylen}"/>
       </geometry>
-      <origin rpy="0 0 0" xyz="0 0 4.1"/>
+      <origin rpy="0 0 0" xyz="0 0 ${bodylen-joint_offset}"/>
       <material name="blue"/>
     </visual>
